File: rasp_power_module/rasp_power_module.kicad_sch (KiCad schematic)
At the start: 22 parts, among them J1 Conn_01x02, J2 Conn_01x05, J3 Conn_01x02, J5 Conn_01x02, J7 Conn_01x02, J8 Conn_01x02, J9 Conn_01x02, K1 G5V-1, K2 FINDER-36.11, Q1 BC847

Commit message: rasp_power_module smt 관련 작업 추가 및 monitor_control_board 개선
Signed-off-by: Ju, Gyeong-min <jcmh74@gmail.com>
Parts:
- D1: value ZMM5V1 -> ZMM5V6-M
- Q1: value BC847 -> S8050 J3Y
Changed lines of the file:
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@@
     (in_bom yes) (on_board yes)
     (property "Reference" "D1" (id 0) (at 103.505 87.63 0))
-    (property "Value" "ZMM5V1" (id 1) (at 103.505 85.09 0))
+    (property "Value" "ZMM5V6-M" (id 1) (at 103.505 85.09 0))
     (property "Footprint" "Diode_SMD:D_MiniMELF" (id 2) (at 103.505 85.725 0)
       (effects (font (size 1.27 1.27)) hide)
@@
       (effects (font (size 1.27 1.27)) (justify left))
     )
-    (property "Value" "BC847" (id 1) (at 91.44 106.0449 0)
+    (property "Value" "S8050 J3Y" (id 1) (at 91.44 106.0449 0)
       (effects (font (size 1.27 1.27)) (justify left))
     )
@@
     )
     (path "/6ffa32bb-1b7b-4bd8-8ba6-9a0e1e29d446"
-      (reference "D1") (unit 1) (value "ZMM5V1") (footprint "Diode_SMD:D_MiniMELF")
+      (reference "D1") (unit 1) (value "ZMM5V6-M") (footprint "Diode_SMD:D_MiniMELF")
     )
     (path "/da01d749-a415-47cd-ace4-8856b376a7d1"
@@
     )
     (path "/d84b1815-2690-4690-8b03-9413b97ff56a"
-      (reference "Q1") (unit 1) (value "BC847") (footprint "Package_TO_SOT_SMD:SOT-23")
+      (reference "Q1") (unit 1) (value "S8050 J3Y") (footprint "Package_TO_SOT_SMD:SOT-23")
     )
     (path "/9931a1f5-893c-49a1-984f-e907ea5ea560"

Commit message: rasp-power-module 마커 변경
Signed-off-by: Ju, Gyeong-min <jcmh74@gmail.com>
Connections:
- net POWER_SIG: now also J3.2 (Pin_2), R1.1; no longer J3.1 (Pin_1), R3.2, R4.2
- net SHUTDOWN: now also J3.1 (Pin_1), R3.2, R4.2; no longer J3.2 (Pin_2), R1.1
Changed lines of the file:
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@@
     (effects (font (size 1.27 1.27)) (justify left bottom))
   )
-  (label "POWER_SIG" (at 194.945 113.03 180)
+  (label "SHUTDOWN" (at 194.945 113.03 180)
     (effects (font (size 1.27 1.27)) (justify right bottom))
   )
-  (label "SHUTDOWN" (at 194.945 115.57 180)
+  (label "POWER_SIG" (at 194.945 115.57 180)
     (effects (font (size 1.27 1.27)) (justify right bottom))
   )

Commit message: rev.2 버전업
Signed-off-by: Ju, Gyeong-min <jcmh74@gmail.com>
Other:
- company: (none) -> for game machine makers
- title: (none) -> Raspberry Pie Power Module
Changed lines of the file:
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@@
 (kicad_sch (version 20211123) (generator eeschema)
   (paper "A4")
+  (title_block
+    (title "Raspberry Pie Power Module")
+    (date "2023-01-11")
+    (rev "2")
+    (company "for game machine makers")
+  )
   (junction (at 114.935 162.56) (diameter 0) (color 0 0 0 0)
   )

Commit message: rasp_pm의 MP1584 모듈 실측치 적용
Signed-off-by: Ju, Gyeong-min <jcmh74@gmail.com>
Parts:
- J1: footprint Connector_Wire:SolderWire-2sqmm_1x02_P7.8mm_D2mm_OD3.9mm -> Connector_Wire:SolderWire-1.5sqmm_1x02_P7.8mm_D1.7mm_OD3.9mm
- J5: footprint Connector_Wire:SolderWire-1.5sqmm_1x02_P7.8mm_D1.7mm_OD3.9mm -> Connector_Wire:SolderWire-1.5sqmm_1x02_P6mm_D1.7mm_OD3mm
Changed lines of the file:
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@@
     (property "Reference" "J1" (id 0) (at 29.845 51.435 0))
     (property "Value" "Conn_01x02" (id 1) (at 29.845 53.975 0))
-    (property "Footprint" "Connector_Wire:SolderWire-2sqmm_1x02_P7.8mm_D2mm_OD3.9mm" (id 2) (at 29.845 57.785 0)
+    (property "Footprint" "Connector_Wire:SolderWire-1.5sqmm_1x02_P7.8mm_D1.7mm_OD3.9mm" (id 2) (at 29.845 57.785 0)
       (effects (font (size 1.27 1.27)) hide)
     )
@@
       (effects (font (size 1.27 1.27)) (justify left))
     )
-    (property "Footprint" "Connector_Wire:SolderWire-1.5sqmm_1x02_P7.8mm_D1.7mm_OD3.9mm" (id 2) (at 38.735 168.91 0)
+    (property "Footprint" "Connector_Wire:SolderWire-1.5sqmm_1x02_P6mm_D1.7mm_OD3mm" (id 2) (at 38.735 168.91 0)
       (effects (font (size 1.27 1.27)) hide)
     )
@@
     )
     (path "/5a04342f-e4df-44b9-ba51-298c1cfa0d1d"
-      (reference "J1") (unit 1) (value "Conn_01x02") (footprint "Connector_Wire:SolderWire-2sqmm_1x02_P7.8mm_D2mm_OD3.9mm")
+      (reference "J1") (unit 1) (value "Conn_01x02") (footprint "Connector_Wire:SolderWire-1.5sqmm_1x02_P7.8mm_D1.7mm_OD3.9mm")
     )
     (path "/0fb0e148-7e8a-4b3c-b734-94d642398d1c"
@@
     )
     (path "/d66a6e59-d578-47f3-99d4-f797be9d6a2a"
-      (reference "J5") (unit 1) (value "Conn_01x02") (footprint "Connector_Wire:SolderWire-1.5sqmm_1x02_P7.8mm_D1.7mm_OD3.9mm")
+      (reference "J5") (unit 1) (value "Conn_01x02") (footprint "Connector_Wire:SolderWire-1.5sqmm_1x02_P6mm_D1.7mm_OD3mm")
     )
     (path "/44853d00-3f66-4577-b2c7-73415bd36cf1"

Commit message: rasp_pm의 smd 부품을 0603에서 0805로 변경
Signed-off-by: Ju, Gyeong-min <jcmh74@gmail.com>
Parts:
- D3: footprint LED_SMD:LED_0603_1608Metric -> LED_SMD:LED_0805_2012Metric
- R1, R2, R3, R4, R5: footprint Resistor_SMD:R_0603_1608Metric -> Resistor_SMD:R_0805_2012Metric
Changed lines of the file:
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@@
       (effects (font (size 1.27 1.27)) (justify right))
     )
-    (property "Footprint" "LED_SMD:LED_0603_1608Metric" (id 2) (at 157.48 138.43 0)
+    (property "Footprint" "LED_SMD:LED_0805_2012Metric" (id 2) (at 157.48 138.43 0)
       (effects (font (size 1.27 1.27)) hide)
     )
@@
     (property "Reference" "R2" (id 0) (at 111.76 104.14 90))
     (property "Value" "10K" (id 1) (at 111.76 106.68 90))
-    (property "Footprint" "Resistor_SMD:R_0603_1608Metric" (id 2) (at 111.506 110.236 90)
+    (property "Footprint" "Resistor_SMD:R_0805_2012Metric" (id 2) (at 111.506 110.236 90)
       (effects (font (size 1.27 1.27)) hide)
     )
@@
     (property "Reference" "R1" (id 0) (at 111.76 95.885 90))
     (property "Value" "1K" (id 1) (at 111.76 98.425 90))
-    (property "Footprint" "Resistor_SMD:R_0603_1608Metric" (id 2) (at 111.506 101.981 90)
+    (property "Footprint" "Resistor_SMD:R_0805_2012Metric" (id 2) (at 111.506 101.981 90)
       (effects (font (size 1.27 1.27)) hide)
     )
@@
     (property "Reference" "R3" (id 0) (at 168.275 86.995 90))
     (property "Value" "100K" (id 1) (at 168.275 89.535 90))
-    (property "Footprint" "Resistor_SMD:R_0603_1608Metric" (id 2) (at 168.529 91.059 90)
+    (property "Footprint" "Resistor_SMD:R_0805_2012Metric" (id 2) (at 168.529 91.059 90)
       (effects (font (size 1.27 1.27)) hide)
     )
@@
     (property "Reference" "R5" (id 0) (at 167.64 133.35 90))
     (property "Value" "4K7" (id 1) (at 167.64 135.89 90))
-    (property "Footprint" "Resistor_SMD:R_0603_1608Metric" (id 2) (at 167.386 139.446 90)
+    (property "Footprint" "Resistor_SMD:R_0805_2012Metric" (id 2) (at 167.386 139.446 90)
       (effects (font (size 1.27 1.27)) hide)
     )
@@
     (property "Reference" "R4" (id 0) (at 168.275 95.25 90))
     (property "Value" "30K" (id 1) (at 168.275 97.79 90))
-    (property "Footprint" "Resistor_SMD:R_0603_1608Metric" (id 2) (at 168.529 99.314 90)
+    (property "Footprint" "Resistor_SMD:R_0805_2012Metric" (id 2) (at 168.529 99.314 90)
       (effects (font (size 1.27 1.27)) hide)
     )
@@
     )
     (path "/2d7a1a59-7c3b-4322-8062-cc884281e53c"
-      (reference "D3") (unit 1) (value "LED") (footprint "LED_SMD:LED_0603_1608Metric")
+      (reference "D3") (unit 1) (value "LED") (footprint "LED_SMD:LED_0805_2012Metric")
     )
     (path "/8a68d06e-7677-429c-9d3e-6573c59f9599"
@@
     )
     (path "/9931a1f5-893c-49a1-984f-e907ea5ea560"
-      (reference "R1") (unit 1) (value "1K") (footprint "Resistor_SMD:R_0603_1608Metric")
+      (reference "R1") (unit 1) (value "1K") (footprint "Resistor_SMD:R_0805_2012Metric")
     )
     (path "/3393e045-4324-474d-9912-cc071730c52a"
-      (reference "R2") (unit 1) (value "10K") (footprint "Resistor_SMD:R_0603_1608Metric")
+      (reference "R2") (unit 1) (value "10K") (footprint "Resistor_SMD:R_0805_2012Metric")
     )
     (path "/b363bb50-dd92-41bf-b98e-38ae28943b4b"
-      (reference "R3") (unit 1) (value "100K") (footprint "Resistor_SMD:R_0603_1608Metric")
+      (reference "R3") (unit 1) (value "100K") (footprint "Resistor_SMD:R_0805_2012Metric")
     )
     (path "/f137e43c-cd03-4192-b5ec-59d668611dd9"
-      (reference "R4") (unit 1) (value "30K") (footprint "Resistor_SMD:R_0603_1608Metric")
+      (reference "R4") (unit 1) (value "30K") (footprint "Resistor_SMD:R_0805_2012Metric")
     )
     (path "/e221d7fe-36ff-4fb6-8a9e-76472ef4a25d"
-      (reference "R5") (unit 1) (value "4K7") (footprint "Resistor_SMD:R_0603_1608Metric")
-    )
-  )
+      (reference "R5") (unit 1) (value "4K7") (footprint "Resistor_SMD:R_0805_2012Metric")
+    )
+  )

Commit message: rasp_pm 다이오드 교체
Signed-off-by: Ju, Gyeong-min <jcmh74@gmail.com>
Parts:
- D1: value ZMM5V6-M -> 1N4148; footprint Diode_SMD:D_MiniMELF -> Diode_THT:D_DO-35_SOD27_P7.62mm_Horizontal; symbol Diode:ZMMxx -> Diode:1N4148
- D2: value 1N4001 -> 1N4007; footprint Diode_SMD:D_SMC-RM10_Universal_Handsoldering -> Diode_THT:D_DO-41_SOD81_P10.16mm_Horizontal; symbol Diode:1N4001 -> Diode:1N4007
Changed lines of the file:
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@@
     (pin "A2")
   )
-  (symbol (lib_id "Diode:ZMMxx") (at 103.505 81.28 0) (mirror y) (unit 1)
+  (symbol (lib_id "Diode:1N4148") (at 103.505 81.28 0) (mirror y) (unit 1)
     (in_bom yes) (on_board yes)
     (property "Reference" "D1" (id 0) (at 103.505 87.63 0))
-    (property "Value" "ZMM5V6-M" (id 1) (at 103.505 85.09 0))
-    (property "Footprint" "Diode_SMD:D_MiniMELF" (id 2) (at 103.505 85.725 0)
-      (effects (font (size 1.27 1.27)) hide)
-    )
-    (property "Datasheet" "https://diotec.com/tl_files/diotec/files/pdf/datasheets/zmm1.pdf" (id 3) (at 103.505 81.28 0)
+    (property "Value" "1N4148" (id 1) (at 103.505 85.09 0))
+    (property "Footprint" "Diode_THT:D_DO-35_SOD27_P7.62mm_Horizontal" (id 2) (at 103.505 81.28 0)
+      (effects (font (size 1.27 1.27)) hide)
+    )
+    (property "Datasheet" "https://assets.nexperia.com/documents/data-sheet/1N4148_1N4448.pdf" (id 3) (at 103.505 81.28 0)
       (effects (font (size 1.27 1.27)) hide)
     )
@@
     (pin "3")
   )
-  (symbol (lib_id "Diode:1N4001") (at 140.335 86.36 90) (mirror x) (unit 1)
+  (symbol (lib_id "Diode:1N4007") (at 140.335 86.36 90) (mirror x) (unit 1)
     (in_bom yes) (on_board yes) (fields_autoplaced)
     (property "Reference" "D2" (id 0) (at 142.875 85.0899 90)
       (effects (font (size 1.27 1.27)) (justify right))
     )
-    (property "Value" "1N4001" (id 1) (at 142.875 87.6299 90)
+    (property "Value" "1N4007" (id 1) (at 142.875 87.6299 90)
       (effects (font (size 1.27 1.27)) (justify right))
     )
-    (property "Footprint" "Diode_SMD:D_SMC-RM10_Universal_Handsoldering" (id 2) (at 140.335 86.36 0)
+    (property "Footprint" "Diode_THT:D_DO-41_SOD81_P10.16mm_Horizontal" (id 2) (at 144.78 86.36 0)
       (effects (font (size 1.27 1.27)) hide)
     )
@@
     )
     (path "/6ffa32bb-1b7b-4bd8-8ba6-9a0e1e29d446"
-      (reference "D1") (unit 1) (value "ZMM5V6-M") (footprint "Diode_SMD:D_MiniMELF")
+      (reference "D1") (unit 1) (value "1N4148") (footprint "Diode_THT:D_DO-35_SOD27_P7.62mm_Horizontal")
     )
     (path "/da01d749-a415-47cd-ace4-8856b376a7d1"
-      (reference "D2") (unit 1) (value "1N4001") (footprint "Diode_SMD:D_SMC-RM10_Universal_Handsoldering")
+      (reference "D2") (unit 1) (value "1N4007") (footprint "Diode_THT:D_DO-41_SOD81_P10.16mm_Horizontal")
     )
     (path "/2d7a1a59-7c3b-4322-8062-cc884281e53c"

Commit message: rasp_pm 다이오드 부품 교체
Signed-off-by: Ju, Gyeong-min <jcmh74@gmail.com>
Parts:
- D1: value 1N4148 -> LL4148; footprint Diode_THT:D_DO-35_SOD27_P7.62mm_Horizontal -> Diode_SMD:D_MiniMELF; symbol Diode:1N4148 -> Diode:LL4148
Changed lines of the file:
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@@
     (pin "A2")
   )
-  (symbol (lib_id "Diode:1N4148") (at 103.505 81.28 0) (mirror y) (unit 1)
+  (symbol (lib_id "Diode:LL4148") (at 103.505 81.28 0) (mirror y) (unit 1)
     (in_bom yes) (on_board yes)
     (property "Reference" "D1" (id 0) (at 103.505 87.63 0))
-    (property "Value" "1N4148" (id 1) (at 103.505 85.09 0))
-    (property "Footprint" "Diode_THT:D_DO-35_SOD27_P7.62mm_Horizontal" (id 2) (at 103.505 81.28 0)
-      (effects (font (size 1.27 1.27)) hide)
-    )
-    (property "Datasheet" "https://assets.nexperia.com/documents/data-sheet/1N4148_1N4448.pdf" (id 3) (at 103.505 81.28 0)
+    (property "Value" "LL4148" (id 1) (at 103.505 85.09 0))
+    (property "Footprint" "Diode_SMD:D_MiniMELF" (id 2) (at 103.505 85.725 0)
+      (effects (font (size 1.27 1.27)) hide)
+    )
+    (property "Datasheet" "http://www.vishay.com/docs/85557/ll4148.pdf" (id 3) (at 103.505 81.28 0)
       (effects (font (size 1.27 1.27)) hide)
     )
@@
     )
     (path "/6ffa32bb-1b7b-4bd8-8ba6-9a0e1e29d446"
-      (reference "D1") (unit 1) (value "1N4148") (footprint "Diode_THT:D_DO-35_SOD27_P7.62mm_Horizontal")
+      (reference "D1") (unit 1) (value "LL4148") (footprint "Diode_SMD:D_MiniMELF")
     )
     (path "/da01d749-a415-47cd-ace4-8856b376a7d1"

Commit message: rasp_pi 다이오드 교체
Signed-off-by: Ju, Gyeong-min <jcmh74@gmail.com>
Parts:
- D2: footprint Diode_THT:D_DO-41_SOD81_P10.16mm_Horizontal -> Diode_SMD:D_SMC-RM10_Universal_Handsoldering
Changed lines of the file:
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@@
       (effects (font (size 1.27 1.27)) (justify right))
     )
-    (property "Footprint" "Diode_THT:D_DO-41_SOD81_P10.16mm_Horizontal" (id 2) (at 144.78 86.36 0)
+    (property "Footprint" "Diode_SMD:D_SMC-RM10_Universal_Handsoldering" (id 2) (at 144.78 86.36 0)
       (effects (font (size 1.27 1.27)) hide)
     )
@@
     )
     (path "/da01d749-a415-47cd-ace4-8856b376a7d1"
-      (reference "D2") (unit 1) (value "1N4007") (footprint "Diode_THT:D_DO-41_SOD81_P10.16mm_Horizontal")
+      (reference "D2") (unit 1) (value "1N4007") (footprint "Diode_SMD:D_SMC-RM10_Universal_Handsoldering")
     )
     (path "/2d7a1a59-7c3b-4322-8062-cc884281e53c"
