File: rasp_power_module/rasp_power_module.kicad_sch (KiCad schematic)
At the start: 22 parts, among them J1 Conn_01x02, J2 Conn_01x05, J3 Conn_01x02, J5 Conn_01x02, J7 Conn_01x02, J8 Conn_01x02, J9 Conn_01x02, K1 G5V-1, K2 FINDER-36.11, Q1 S8050 J3Y

Commit message: rasp_pm 릴레이 종류 변경
Signed-off-by: Ju, Gyeong-min <jcmh74@gmail.com>
Parts:
- removed K2: FINDER-36.11, Relay_THT:Relay_SPDT_Finder_36.11, symbol Relay:FINDER-36.11
- added K2: SANYOU_SRD_Form_C, Relay_THT:Relay_SPDT_SANYOU_SRD_Series_Form_C, symbol Relay:SANYOU_SRD_Form_C
Connections:
- net +12V: now also K2.1
- net 12V_ON: now also K2.3
- net 5V_ON: now also K2.5
- net Relay_Coil_2: now also K2.2
Changed lines of the file:
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@@
   )
   (no_connect (at 248.92 38.1))
-  (no_connect (at 248.92 71.12))
+  (no_connect (at 233.68 71.12))
   (wire (pts (xy 123.825 41.91) (xy 123.825 55.245))
     (stroke (width 0) (type default) (color 0 0 0 0))
@@
     )
   )
-  (global_label "Relay_In" (shape input) (at 233.68 68.58 180) (fields_autoplaced)
+  (global_label "Relay_In" (shape input) (at 248.92 68.58 0) (fields_autoplaced)
+    (effects (font (size 1.27 1.27)) (justify left))
+    (property "Intersheet References" "${INTERSHEET_REFS}" (id 0) (at 259.195 68.5006 0)
+      (effects (font (size 1.27 1.27)) (justify left) hide)
+    )
+  )
+  (global_label "12V_ON" (shape input) (at 123.825 40.005 90) (fields_autoplaced)
+    (effects (font (size 1.27 1.27)) (justify left))
+    (property "Intersheet References" "${INTERSHEET_REFS}" (id 0) (at 123.7456 30.4557 90)
+      (effects (font (size 1.27 1.27)) (justify left) hide)
+    )
+  )
+  (global_label "OutVCC" (shape input) (at 252.095 108.585 0) (fields_autoplaced)
+    (effects (font (size 1.27 1.27)) (justify left))
+    (property "Intersheet References" "${INTERSHEET_REFS}" (id 0) (at 261.3419 108.6644 0)
+      (effects (font (size 1.27 1.27)) (justify left) hide)
+    )
+  )
+  (global_label "12V_ON" (shape input) (at 71.755 127 0) (fields_autoplaced)
+    (effects (font (size 1.27 1.27)) (justify left))
+    (property "Intersheet References" "${INTERSHEET_REFS}" (id 0) (at 81.3043 126.9206 0)
+      (effects (font (size 1.27 1.27)) (justify left) hide)
+    )
+  )
+  (global_label "Relay_Coil_2" (shape input) (at 248.92 78.74 0) (fields_autoplaced)
+    (effects (font (size 1.27 1.27)) (justify left))
+    (property "Intersheet References" "${INTERSHEET_REFS}" (id 0) (at 263.3074 78.6606 0)
+      (effects (font (size 1.27 1.27)) (justify left) hide)
+    )
+  )
+  (global_label "5V_ON" (shape input) (at 71.755 137.795 0) (fields_autoplaced)
+    (effects (font (size 1.27 1.27)) (justify left))
+    (property "Intersheet References" "${INTERSHEET_REFS}" (id 0) (at 80.0948 137.7156 0)
+      (effects (font (size 1.27 1.27)) (justify left) hide)
+    )
+  )
+  (global_label "5V_ON" (shape input) (at 142.24 160.02 0) (fields_autoplaced)
+    (effects (font (size 1.27 1.27)) (justify left))
+    (property "Intersheet References" "${INTERSHEET_REFS}" (id 0) (at 150.5798 159.9406 0)
+      (effects (font (size 1.27 1.27)) (justify left) hide)
+    )
+  )
+  (global_label "Relay_Out" (shape input) (at 233.68 66.04 180) (fields_autoplaced)
     (effects (font (size 1.27 1.27)) (justify right))
-    (property "Intersheet References" "${INTERSHEET_REFS}" (id 0) (at 223.405 68.5006 0)
+    (property "Intersheet References" "${INTERSHEET_REFS}" (id 0) (at 221.9536 65.9606 0)
       (effects (font (size 1.27 1.27)) (justify right) hide)
-    )
-  )
-  (global_label "12V_ON" (shape input) (at 123.825 40.005 90) (fields_autoplaced)
-    (effects (font (size 1.27 1.27)) (justify left))
-    (property "Intersheet References" "${INTERSHEET_REFS}" (id 0) (at 123.7456 30.4557 90)
-      (effects (font (size 1.27 1.27)) (justify left) hide)
-    )
-  )
-  (global_label "OutVCC" (shape input) (at 252.095 108.585 0) (fields_autoplaced)
-    (effects (font (size 1.27 1.27)) (justify left))
-    (property "Intersheet References" "${INTERSHEET_REFS}" (id 0) (at 261.3419 108.6644 0)
-      (effects (font (size 1.27 1.27)) (justify left) hide)
-    )
-  )
-  (global_label "12V_ON" (shape input) (at 71.755 127 0) (fields_autoplaced)
-    (effects (font (size 1.27 1.27)) (justify left))
-    (property "Intersheet References" "${INTERSHEET_REFS}" (id 0) (at 81.3043 126.9206 0)
-      (effects (font (size 1.27 1.27)) (justify left) hide)
-    )
-  )
-  (global_label "Relay_Coil_2" (shape input) (at 248.92 78.74 0) (fields_autoplaced)
-    (effects (font (size 1.27 1.27)) (justify left))
-    (property "Intersheet References" "${INTERSHEET_REFS}" (id 0) (at 263.3074 78.6606 0)
-      (effects (font (size 1.27 1.27)) (justify left) hide)
-    )
-  )
-  (global_label "5V_ON" (shape input) (at 71.755 137.795 0) (fields_autoplaced)
-    (effects (font (size 1.27 1.27)) (justify left))
-    (property "Intersheet References" "${INTERSHEET_REFS}" (id 0) (at 80.0948 137.7156 0)
-      (effects (font (size 1.27 1.27)) (justify left) hide)
-    )
-  )
-  (global_label "5V_ON" (shape input) (at 142.24 160.02 0) (fields_autoplaced)
-    (effects (font (size 1.27 1.27)) (justify left))
-    (property "Intersheet References" "${INTERSHEET_REFS}" (id 0) (at 150.5798 159.9406 0)
-      (effects (font (size 1.27 1.27)) (justify left) hide)
-    )
-  )
-  (global_label "Relay_Out" (shape input) (at 248.92 66.04 0) (fields_autoplaced)
-    (effects (font (size 1.27 1.27)) (justify left))
-    (property "Intersheet References" "${INTERSHEET_REFS}" (id 0) (at 260.6464 65.9606 0)
-      (effects (font (size 1.27 1.27)) (justify left) hide)
     )
   )
@@
     (pin "1")
   )
+  (symbol (lib_id "Relay:SANYOU_SRD_Form_C") (at 241.3 73.66 90) (unit 1)
+    (in_bom yes) (on_board yes) (fields_autoplaced)
+    (property "Reference" "K2" (id 0) (at 241.3 58.42 90))
+    (property "Value" "SANYOU_SRD_Form_C" (id 1) (at 241.3 60.96 90))
+    (property "Footprint" "Relay_THT:Relay_SPDT_SANYOU_SRD_Series_Form_C" (id 2) (at 242.57 62.23 0)
+      (effects (font (size 1.27 1.27)) (justify left) hide)
+    )
+    (property "Datasheet" "http://www.sanyourelay.ca/public/products/pdf/SRD.pdf" (id 3) (at 241.3 73.66 0)
+      (effects (font (size 1.27 1.27)) hide)
+    )
+    (pin "1")
+    (pin "2")
+    (pin "3")
+    (pin "4")
+    (pin "5")
+  )
   (symbol (lib_id "Connector_Generic:Conn_01x05") (at 31.115 92.075 0) (mirror y) (unit 1)
     (in_bom yes) (on_board yes) (fields_autoplaced)
@@
     (pin "2")
   )
-  (symbol (lib_id "Relay:FINDER-36.11") (at 241.3 73.66 270) (mirror x) (unit 1)
-    (in_bom yes) (on_board yes) (fields_autoplaced)
-    (property "Reference" "K2" (id 0) (at 241.3 58.42 90))
-    (property "Value" "FINDER-36.11" (id 1) (at 241.3 60.96 90))
-    (property "Footprint" "Relay_THT:Relay_SPDT_Finder_36.11" (id 2) (at 240.538 41.402 0)
-      (effects (font (size 1.27 1.27)) hide)
-    )
-    (property "Datasheet" "https://gfinder.findernet.com/public/attachments/36/EN/S36EN.pdf" (id 3) (at 241.3 73.66 0)
-      (effects (font (size 1.27 1.27)) hide)
-    )
-    (pin "11")
-    (pin "12")
-    (pin "14")
-    (pin "A1")
-    (pin "A2")
-  )
   (symbol (lib_id "Diode:LL4148") (at 103.505 81.28 0) (mirror y) (unit 1)
     (in_bom yes) (on_board yes)
@@
       (reference "K1") (unit 1) (value "G5V-1") (footprint "Relay_THT:Relay_SPDT_Omron_G5V-1")
     )
-    (path "/6dd969ac-f79d-4c56-98be-25fb6ceb6df2"
-      (reference "K2") (unit 1) (value "FINDER-36.11") (footprint "Relay_THT:Relay_SPDT_Finder_36.11")
+    (path "/0ea7957c-a5a7-4d62-b5d7-ca3967a7f783"
+      (reference "K2") (unit 1) (value "SANYOU_SRD_Form_C") (footprint "Relay_THT:Relay_SPDT_SANYOU_SRD_Series_Form_C")
     )
     (path "/d84b1815-2690-4690-8b03-9413b97ff56a"
