File: battery_array/battery_array.kicad_sch (KiCad schematic)
At the start: 68 parts, among them J1 Conn_01x02_Male, J10 Conn_01x02_Male, J11 Conn_01x02_Male, J12 Conn_01x02_Male, J13 Conn_01x02_Male, J14 Conn_01x02_Male, J15 Conn_01x02_Male, J16 Conn_01x02_Male, J17 Conn_01x02_Male, J18 Conn_01x02_Male, J19 Conn_01x02_Male, J2 Conn_01x02_Male, J20 Conn_01x02_Male, J21 Conn_01x02_Male, J22 Conn_01x02_Male, J23 Conn_01x02_Male, J24 Conn_01x02_Male, J25 Conn_01x02_Male, J26 Conn_01x02_Male, J27 Conn_01x02_Male, J28 Conn_01x02_Male, J29 Conn_01x02_Male, J3 Conn_01x02_Male, J30 Conn_01x02_Male, J31 Conn_01x02_Male, J32 Conn_01x02_Male, J33 Conn_01x02_Male, J34 Conn_01x02_Male, J35 Conn_01x02_Male, J36 Conn_01x02_Male, J37 Conn_01x02_Male, J38 Conn_01x02_Male, J39 Conn_01x02_Male, J4 Conn_01x02_Male, J40 Conn_01x02_Male, J41 Conn_01x02_Male, J42 Conn_01x02_Male, J43 Conn_01x02_Male, J44 Conn_01x02_Male, J45 Conn_01x02_Male, J46 Conn_01x02_Male, J47 Conn_01x02_Male, J48 Conn_01x02_Male, J49 Conn_01x02_Male, J5 Conn_01x02_Male, J50 Conn_01x02_Male, J51 Conn_01x02_Male, J52 Conn_01x02_Male, J53 Conn_01x02_Male, J54 Conn_01x02_Male, J55 Conn_01x02_Male, J56 Conn_01x02_Male, J57 Conn_01x02_Male, J58 Conn_01x02_Male, J59 Conn_01x02_Male, J6 Conn_01x02_Male, J60 Conn_01x02_Male, J7 Conn_01x02_Male, J8 Conn_01x02_Male, J9 Conn_01x02_Male

Commit message: 도면 시트 설명 추가
Signed-off-by: Ju, Gyeong-min <jcmh74@gmail.com>
Other:
- company: (none) -> Amos Home
- title: (none) -> Amos 3S20P Battery Array Board
Changed lines of the file:
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@@
 (kicad_sch (version 20211123) (generator eeschema)
   (paper "A4")
+  (title_block
+    (title "Amos 3S20P Battery Array Board")
+    (rev "1")
+    (company "Amos Home")
+  )
   (junction (at 58.42 30.48) (diameter 0) (color 0 0 0 0)
   )
