File: input-74hc165/input-74hc165.kicad_sch (KiCad schematic)
At the start: 6 parts, among them J1 Conn_01x10_Male

Commit message: 도면 시트 설명 추가
Signed-off-by: Ju, Gyeong-min <jcmh74@gmail.com>
Other:
- company: (none) -> Amos Home
- title: (none) -> 74HC165 Input Board
Changed lines of the file:
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@@
 (kicad_sch (version 20211123) (generator eeschema)
   (paper "A4")
+  (title_block
+    (title "74HC165 Input Board")
+    (rev "1")
+    (company "Amos Home")
+  )
   (junction (at 194.31 41.91) (diameter 0) (color 0 0 0 0)
   )
