File: joystick-input/joystick-input.kicad_sch (KiCad schematic)
At the start: 11 parts, among them J1 Conn_01x18_Male

Commit message: 도면 시트 설명 추가
Signed-off-by: Ju, Gyeong-min <jcmh74@gmail.com>
Other:
- company: (none) -> Amos Home
- title: (none) -> Joystick Input Board
Changed lines of the file:
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@@
 (kicad_sch (version 20211123) (generator eeschema)
   (paper "A4")
+  (title_block
+    (title "Joystick Input Board")
+    (rev "2")
+    (company "Amos Home")
+  )
   (junction (at 229.87 48.26) (diameter 0) (color 0 0 0 0)
   )
