File: joystick-input_jst/joystick-input.kicad_sch (KiCad schematic)
At the start: 38 parts, among them J11 Conn_01x05, J12 Conn_01x02, J13 Conn_01x02, J14 Conn_01x02, J15 Conn_01x02, J16 Conn_01x02, J17 Conn_01x02, J18 Conn_01x02, J19 Conn_01x02, J21 Conn_01x05, J22 Conn_01x02, J23 Conn_01x02, J24 Conn_01x02, J25 Conn_01x02, J26 Conn_01x02, J27 Conn_01x02, J28 Conn_01x02, J29 Conn_01x02

Commit message: 도면 시트 설명 추가
Signed-off-by: Ju, Gyeong-min <jcmh74@gmail.com>
Other:
- company: (none) -> Amos Home
- title: (none) -> Joystick Input (JST Ver)
Changed lines of the file:
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@@
 (kicad_sch (version 20211123) (generator eeschema)
   (paper "A4")
+  (title_block
+    (title "Joystick Input (JST Ver)")
+    (rev "1")
+    (company "Amos Home")
+  )
   (junction (at 173.99 74.93) (diameter 0) (color 0 0 0 0)
   )
