File: odroid-extend/odroid-extend.kicad_pcb (KiCad board)
At the start: 2 copper layers, 58.4 x 65.5 mm, 7 parts, among them J1 Conn_02x20_Odd_Even, J2 Conn_01x20_Male, J3 Conn_01x20_Male, J4 Conn_01x02_Male, J5 Conn_01x02_Male, J6 Conn_01x02_Male, J7 Conn_01x02_Male

Commit message: kicad 6으로 마이그레이션
Signed-off-by: Ju, Gyeong-min <jcmh74@gmail.com>
Other:
- net class Default removed
