File: odroid-extend/odroid-extend.kicad_sch (KiCad schematic)
At the start: 7 parts, among them J1 Conn_02x20_Odd_Even, J2 Conn_01x20_Male, J3 Conn_01x20_Male, J4 Conn_01x02_Male, J5 Conn_01x02_Male, J6 Conn_01x02_Male, J7 Conn_01x02_Male

Commit message: 도면 시트 설명 추가
Signed-off-by: Ju, Gyeong-min <jcmh74@gmail.com>
Other:
- company: (none) -> Amos Home
- title: (none) -> Odroid N2(+) GPIO Extend Board
Changed lines of the file:
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@@
 (kicad_sch (version 20211123) (generator eeschema)
   (paper "A4")
+  (title_block
+    (title "Odroid N2(+) GPIO Extend Board")
+    (rev "1")
+    (company "Amos Home")
+  )
   (junction (at 127 82.55) (diameter 0) (color 0 0 0 0)
   )
