File: esp-prog-adaptor/esp-prog-adator.kicad_sch (KiCad schematic)
At the start: 6 parts, among them J1 Conn_02x19_Odd_Even, J2 Conn_02x19_Odd_Even, J5 Conn_01x03_Male, J6 Conn_01x03_Male

Commit message: 도면 시트 설명 추가
Signed-off-by: Ju, Gyeong-min <jcmh74@gmail.com>
Other:
- company: (none) -> Amos Home
Changed lines of the file:
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@@
     (title "ESP32 JTAG Adapter")
     (date "2021-09-02")
-    (rev "1.0")
+    (rev "2")
+    (company "Amos Home")
     (comment 1 "/blob/master/docs/en/hw-reference/ESP-Prog_guide.rst")
     (comment 2 "https://github.com/espressif/esp-iot-solution")

Commit message: esp_prog_adaptor에 나사홀 추가
Signed-off-by: Ju, Gyeong-min <jcmh74@gmail.com>
Other:
- title: ESP32 JTAG Adapter -> ESP32 JTAG Adapter (for ESP32-DevKitC)
Changed lines of the file:
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@@
   (paper "A4")
   (title_block
-    (title "ESP32 JTAG Adapter")
+    (title "ESP32 JTAG Adapter (for ESP32-DevKitC)")
     (date "2021-09-02")
     (rev "2")
